File: uiuc_ruler.kicad_pcb (KiCad board)
At the start: 2 copper layers, 248.9 x 27.9 mm, 49 parts, among them J2 Barrel_Jack, Q1 TO263/D2PAK, U1 ATtiny85-20PU, U10 SSOP8, U11 TO-252/DPAK, U12 QFP32, U2 LM1117-5.0, U3 SOT23-5, U4 SOT23-3, U5 SOT223, U6 SOIC20, U7 TO220, U8 SOIC8, U9 SOIC14, Y1 Resonator_Small

Commit message: add footprints
Parts:
- removed H1, H2: MountingHole, MountingHole:MountingHole_3.2mm_M3
- removed ISP1: AVR-ISP-6, Connector_IDC:IDC-Header_2x03_P2.54mm_Vertical
- removed J2: Barrel_Jack, Connector_BarrelJack:BarrelJack_CUI_PJ-063AH_Horizontal
- removed RV1: R_POT, Potentiometer_SMD:Potentiometer_Bourns_TC33X_Vertical
- added C2: D8.0mm, uiuc_ruler:cap_d7.5_p3.5, F.Cu at (86.4, 99.1)
- added C3: C_Small, uiuc_ruler:cap_d10_p5, F.Cu at (86.4, 89.5)
- added Q2: SOT-323, Package_TO_SOT_SMD:SOT-323_SC-70, F.Cu at (154.3, 101.6)
- added R20: capacitor_codes, uiuc_ruler:capacitor_codes, F.Cu at (262.9, 89.0)
- added R21: P0.3in, uiuc_ruler:R_Axial_DIN0204_L3.6mm_D1.6mm_P7.62mm_Horizontal, F.Cu at (64.8, 99.1)
- added R22: units, uiuc_ruler:units, F.Cu at (151.1, 93.5)
- added R23: preferrednumbers, uiuc_ruler:preferrednumbers, F.Cu at (226.7, 84.8)
- added R24: P0.5in, uiuc_ruler:R_Axial_DIN0309_L9.0mm_D3.2mm_P12.70mm_Horizontal, F.Cu at (64.8, 99.1)
- added R25: DIP-8, Package_DIP:DIP-8_W8.89mm_SMDSocket_LongPads, F.Cu at (213.4, 88.9)
- added R26: 2010, Resistor_SMD:R_2010_5025Metric, F.Cu at (73.0, 92.7)
- added R27: P0.4in, uiuc_ruler:R_Axial_DIN0207_L6.3mm_D2.5mm_P10.16mm_Horizontal, F.Cu at (64.8, 99.1)
- added R28: resistor_codes, uiuc_ruler:resistor_codes, F.Cu at (276.9, 85.7)
- added RN1: 0402, Resistor_SMD:R_Array_Convex_4x0402, F.Cu at (91.4, 89.0)
- added RN2: 0603, Resistor_SMD:R_Array_Convex_4x0603, F.Cu at (91.4, 93.3)
- added RN3: 1206, Resistor_SMD:R_Array_Convex_4x1206, F.Cu at (91.5, 99.4)
- added SW1: SW-6mm, uiuc_ruler:SW_PUSH_6mm, F.Cu at (243.8, 85.1)
- added SW2: SW-12mm, uiuc_ruler:SW_PUSH-12mm, F.Cu at (240.7, 94.6)
- added U13: SOT-363, Package_TO_SOT_SMD:SOT-363_SC-70-6, F.Cu at (154.9, 97.8)
- added U14: TSSOP-8, Package_SO:TSSOP-8_4.4x3mm_P0.65mm, F.Cu at (218.4, 99.7)
- added U15: SOT-563, Package_TO_SOT_SMD:SOT-563, F.Cu at (175.3, 94.0)
- added U16: QFP-64, Package_QFP:TQFP-64_10x10mm_P0.5mm, F.Cu at (227.3, 90.2)
- added U17: SOT-89, Package_TO_SOT_SMD:SOT-89-3, F.Cu at (175.3, 88.3)
- added Y2: CSTxExxV, Crystal:Resonator_SMD_muRata_CSTxExxV-3Pin_3.0x1.1mm, F.Cu at (127.1, 99.1)
- added Y3: 3.2X2.4, Crystal:Crystal_SMD_3225-4Pin_3.2x2.5mm, F.Cu at (134.2, 100.3)
- added Y4: 5X3.2, Crystal:Crystal_SMD_Qantek_QC5CB-2Pin_5x3.2mm, F.Cu at (127.6, 91.4)
- added Y5: 2.5X2, Crystal:Crystal_SMD_EuroQuartz_X22-4Pin_2.5x2.0mm, F.Cu at (134.0, 95.3)
- added Y6: 2X1.2, Crystal:Crystal_SMD_3215-2Pin_3.2x1.5mm, F.Cu at (134.0, 90.8)
- C1: footprint Capacitor_SMD:C_0805_2012Metric -> uiuc_ruler:cap_d5_p2.5
- D1: value LED -> SOD-123; footprint LED_SMD:LED_0805_2012Metric -> Diode_SMD:D_SOD-123
- D10: value SOD323 -> SOD-323
- D2: value D_Schottky -> SOD-523; footprint Diode_SMD:D_0805_2012Metric -> Diode_SMD:D_SOD-523
- D9: value SOD128 -> SOD-128
- Q1: value TO263/D2PAK -> TO-263
- R1: value R -> awgdrill; footprint Resistor_SMD:R_0805_2012Metric -> uiuc_ruler:awgdrill
- R11: value awgcurrent -> referenceopamp; footprint ece445_pcb:awgcurrent -> uiuc_ruler:referenceopamp
- R12: footprint ece445_pcb:logo -> uiuc_ruler:logo
- R15: footprint ece445_pcb:resistor -> uiuc_ruler:resistor
- R16: footprint ece445_pcb:referencebjt -> uiuc_ruler:referencebjt
- R17: footprint ece445_pcb:referencefet -> uiuc_ruler:referencefet
- R18: footprint ece445_pcb:referencediode -> uiuc_ruler:referencediode
- R19: footprint ece445_pcb:fontsize -> uiuc_ruler:fontsize
- R5: footprint ece445_pcb:rulerinches -> uiuc_ruler:rulerinches
- R6: footprint ece445_pcb:rulercm -> uiuc_ruler:rulercm
- R7: footprint ece445_pcb:traceswidths -> uiuc_ruler:traceswidths
- U1: value ATtiny85-20PU -> QFN-24; footprint Package_SO:SOIC-8_3.9x4.9mm_P1.27mm -> Package_DFN_QFN:QFN-24-1EP_4x4mm_P0.5mm_EP2.6x2.6mm
- U10: value SSOP8 -> BGA-7x7; footprint Package_SO:VSSOP-8_2.3x2mm_P0.5mm -> Package_BGA:VFBGA-49_5.0x5.0mm_Layout7x7_P0.65mm
- U11: value TO-252/DPAK -> TO-252
- U12: value QFP32 -> QFP-32
- U2: value LM1117-5.0 -> VSSOP-8; footprint Package_TO_SOT_SMD:SOT-223 -> Package_SO:VSSOP-8_2.3x2mm_P0.5mm
- U3: value SOT23-5 -> SOT-23-5
- U4: value SOT23-3 -> SOT-23-3
- U5: value SOT223 -> SOT-223
- U6: value SOIC20 -> SOIC-20
- U7: value TO220 -> TO-220; footprint ece445_pcb:TO-220-3_Vertical -> uiuc_ruler:TO-220-3_Vertical
- U8: value SOIC8 -> SOIC-8
- U9: value SOIC14 -> SOIC-14
- Y1: value Resonator_Small -> HC49; footprint Crystal:Resonator-3Pin_W8.0mm_H3.5mm -> Crystal:Crystal_SMD_HC49-SD
- moved R18 175.3 mm to (78.7, 90.8), turned to 180 degrees
- moved R19 172.7 mm to (69.2, 90.2), turned to 90 degrees
- moved R17 170.1 mm to (101.6, 99.1), turned to 0 degrees
- moved R16 169.5 mm to (94.0, 95.2), turned to 180 degrees
- moved R1 154.9 mm to (275.8, 84.8)
- moved R2 92.2 mm to (64.1, 92.7), turned to 90 degrees
- moved R5 91.5 mm to (59.7, 104.1)
- moved D10 89.7 mm to (109.2, 101.0)
- moved R14 88.4 mm to (62.2, 87.0), turned to 90 degrees
- moved U1 88.3 mm to (200.7, 88.3)
- moved R8 87.7 mm to (68.6, 92.7), turned to 90 degrees
- moved U2 86.5 mm to (209.6, 99.7), turned to 0 degrees
- moved R6 86.4 mm to (59.7, 104.1)
- moved R13 84.9 mm to (65.4, 87.0), turned to 90 degrees
- moved D6 84.6 mm to (113.7, 85.1)
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Connections:
- D1 pad 2: /MOSI -> Net-(D1-Pad2)
- D2 pad 1: +5V -> Net-(D2-Pad1)
- U1 pad 1: /~RST -> Net-(U1-Pad1)
- U1 pad 4: GND -> Net-(U1-Pad4)
- U1 pad 5: /MISO -> Net-(U1-Pad5)
- U1 pad 6: /MOSI -> Net-(U1-Pad6)
- U1 pad 7: /SCK -> Net-(U1-Pad7)
- U1 pad 8: +5V -> Net-(U1-Pad8)
- U2 pad 1: GND -> Net-(U2-Pad1)
- U2 pad 2: +5V -> Net-(U2-Pad2)
- U2 pad 4: (no net) -> Net-(U2-Pad4)
- Y1 pad 1: Net-(U1-Pad3) -> Net-(Y1-Pad1)
- Y1 pad 2: GND -> Net-(Y1-Pad2)
Routing:
- net /SCK: track 27.7 -> 0.00 mm
- net +5V: track 18.1 -> 0.00 mm
- net /MOSI: track 17.4 -> 0.00 mm
- net /MISO: track 16.5 -> 0.00 mm, vias 1 -> 0
- net /~RST: track 10.6 -> 0.00 mm
- net Net-(D2-Pad2): track 9.79 -> 0.00 mm
- net Net-(U2-Pad3): track 9.61 -> 0.00 mm
- net Net-(U1-Pad3): track 5.93 -> 0.00 mm
- net Net-(U1-Pad2): track 5.90 -> 0.00 mm
- net Net-(D1-Pad1): track 3.31 -> 0.00 mm
- removed copper zone on B.Cu, net GND
- removed copper zone on F.Cu, net GND
Other:
- board size 248.9 x 27.9 mm -> 259.1 x 27.9 mm
- board text added: "Component Codes"
- board text added: "Oscillators"
- board text added: "RLC"
- board text added: "Switches"
- board text added: "UIUC Ruler V1 Evan Widloski 2021-06-05"
- board text removed: "ECE445 Blinky V1"
- board text removed: "ECE445 Ruler V1 Evan Widloski 2021-06-05"
- board text removed: "RLC - Imperial"
- board text removed: "Team X - 2021-06-03"
