File: uiuc_ruler.kicad_pcb (KiCad board)
At the start: 2 copper layers, 259.1 x 27.9 mm, 71 parts, among them Q1 TO-263, Q2 SOT-323, SW1 SW-6mm, SW2 SW-12mm, U1 QFN-24, U10 BGA-7x7, U11 TO-252, U12 QFP-32, U13 SOT-363, U14 TSSOP-8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

Commit message: add order notes, update resistor/capacitor diagram, add diode label
Parts:
- removed R20: capacitor_codes, uiuc_ruler:capacitor_codes
- removed R28: resistor_codes, uiuc_ruler:resistor_codes
- added REF**: capacitor_codes, uiuc_ruler:capacitor_codes, F.Cu at (262.9, 88.3)
- added REF**: resistor_codes, uiuc_ruler:resistor_codes, F.Cu at (275.0, 90.2)
- R21: value P0.3in -> P7.62mm
- R24: value P0.5in -> P12.7mm
- R27: value P0.4in -> P10.16mm
- moved R15 20.4 mm to (257.8, 82.8), turned to -90 degrees
- moved R23 4.04 mm to (222.7, 84.5)
- moved C1 1.91 mm to (80.5, 94.0)
- moved R1 1.02 mm to (276.9, 84.8)
Other:
- net class Default removed
- board text added: "UIUC Ruler V2 Evan Widloski 2025-02-05"
- board text removed: "UIUC Ruler V1 Evan Widloski 2021-06-05"
