File: uiuc_ruler.sch (KiCad schematic (older format))
At the start: 49 parts, among them J2 Barrel_Jack, Q1 TO263/D2PAK, U1 ATtiny85-20PU, U10 SSOP8, U11 TO-252/DPAK, U12 QFP32, U2 LM1117-5.0, U3 SOT23-5, U4 SOT23-3, U5 SOT223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

Commit message: add footprints
Parts:
- removed D1: LED, LED_SMD:LED_0805_2012Metric, symbol Device:LED
- removed D2: D_Schottky, Diode_SMD:D_0805_2012Metric, symbol Device:D_Schottky
- removed H1, H2: MountingHole, MountingHole:MountingHole_3.2mm_M3, symbol Mechanical:MountingHole
- removed ISP1: AVR-ISP-6, Connector_IDC:IDC-Header_2x03_P2.54mm_Vertical, symbol Connector:AVR-ISP-6
- removed J2: Barrel_Jack, Connector_BarrelJack:BarrelJack_CUI_PJ-063AH_Horizontal, symbol Connector:Barrel_Jack
- removed RV1: R_POT, Potentiometer_SMD:Potentiometer_Bourns_TC33X_Vertical, symbol Device:R_POT
- removed U1: ATtiny85-20PU, Package_SO:SOIC-8_3.9x4.9mm_P1.27mm, symbol MCU_Microchip_ATtiny:ATtiny85-20PU
- removed U10: SSOP8, Package_SO:VSSOP-8_2.3x2mm_P0.5mm, symbol Analog_ADC:ADS7040xDCU
- removed U2: LM1117-5.0, Package_TO_SOT_SMD:SOT-223, symbol Regulator_Linear:LM1117-5.0
- removed Y1: Resonator_Small, Crystal:Resonator-3Pin_W8.0mm_H3.5mm, symbol Device:Resonator_Small
- added C2: D8.0mm, uiuc_ruler:cap_d7.5_p3.5, symbol Device:C_Small
- added C3: C_Small, uiuc_ruler:cap_d10_p5, symbol Device:C_Small
- added D1: SOD-123, Diode_SMD:D_SOD-123, symbol Device:D_Small
- added D2: SOD-523, Diode_SMD:D_SOD-523, symbol Device:D_Small
- added Q2: SOT-323, Package_TO_SOT_SMD:SOT-323_SC-70, symbol Transistor_BJT:2SC4213
- added R20: capacitor_codes, uiuc_ruler:capacitor_codes, symbol Device:R
- added R21: P0.3in, uiuc_ruler:R_Axial_DIN0204_L3.6mm_D1.6mm_P7.62mm_Horizontal, symbol Device:R
- added R22: units, uiuc_ruler:units, symbol Device:R
- added R23: preferrednumbers, uiuc_ruler:preferrednumbers, symbol Device:R
- added R24: P0.5in, uiuc_ruler:R_Axial_DIN0309_L9.0mm_D3.2mm_P12.70mm_Horizontal, symbol Device:R
- added R25: DIP-8, Package_DIP:DIP-8_W8.89mm_SMDSocket_LongPads, symbol Device:R
- added R26: 2010, Resistor_SMD:R_2010_5025Metric, symbol Device:R
- added R27: P0.4in, uiuc_ruler:R_Axial_DIN0207_L6.3mm_D2.5mm_P10.16mm_Horizontal, symbol Device:R
- added R28: resistor_codes, uiuc_ruler:resistor_codes, symbol Device:R
- added RN1: 0402, Resistor_SMD:R_Array_Convex_4x0402, symbol Device:R_Pack04_SIP
- added RN2: 0603, Resistor_SMD:R_Array_Convex_4x0603, symbol Device:R_Pack04_SIP
- added RN3: 1206, Resistor_SMD:R_Array_Convex_4x1206, symbol Device:R_Pack04_SIP
- added SW1: SW-6mm, uiuc_ruler:SW_PUSH_6mm, symbol Switch:SW_Push
- added SW2: SW-12mm, uiuc_ruler:SW_PUSH-12mm, symbol Switch:SW_Push
- added U1: QFN-24, Package_DFN_QFN:QFN-24-1EP_4x4mm_P0.5mm_EP2.6x2.6mm, symbol Analog_ADC:LTC2309_QFN
- added U10: BGA-7x7, Package_BGA:VFBGA-49_5.0x5.0mm_Layout7x7_P0.65mm, symbol MCU_Microchip_ATmega:ATxmega128D4-CU
- added U13: SOT-363, Package_TO_SOT_SMD:SOT-363_SC-70-6, symbol Amplifier_Current:BQ500100DCK
- added U14: TSSOP-8, Package_SO:TSSOP-8_4.4x3mm_P0.65mm, symbol Memory_EEPROM:AT24CS01-XHM
- added U15: SOT-563, Package_TO_SOT_SMD:SOT-563, symbol Logic_LevelTranslator:SN74LVC1T45DRL
- added U16: QFP-64, Package_QFP:TQFP-64_10x10mm_P0.5mm, symbol Analog_ADC:ADS1298xPAG
- added U17: SOT-89, Package_TO_SOT_SMD:SOT-89-3, symbol Regulator_Linear:LM317L_SOT-89
- added U2: VSSOP-8, Package_SO:VSSOP-8_2.3x2mm_P0.5mm, symbol Regulator_Linear:LP2987-3.0_SOIC8_VSSOP8
- added Y1: HC49, Crystal:Crystal_SMD_HC49-SD, symbol Device:Crystal_Small
- added Y2: CSTxExxV, Crystal:Resonator_SMD_muRata_CSTxExxV-3Pin_3.0x1.1mm, symbol Device:Crystal_GND2_Small
- added Y3: 3.2X2.4, Crystal:Crystal_SMD_3225-4Pin_3.2x2.5mm, symbol Device:Crystal_Small
- added Y4: 5X3.2, Crystal:Crystal_SMD_Qantek_QC5CB-2Pin_5x3.2mm, symbol Device:Crystal_Small
- added Y5: 2.5X2, Crystal:Crystal_SMD_EuroQuartz_X22-4Pin_2.5x2.0mm, symbol Device:Crystal_Small
- added Y6: 2X1.2, Crystal:Crystal_SMD_3215-2Pin_3.2x1.5mm, symbol Device:Crystal_Small
- C1: footprint Capacitor_SMD:C_0805_2012Metric -> uiuc_ruler:cap_d5_p2.5
- D10: value SOD323 -> SOD-323
- D9: value SOD128 -> SOD-128
- Q1: value TO263/D2PAK -> TO-263
- R1: value R -> awgdrill; footprint Resistor_SMD:R_0805_2012Metric -> uiuc_ruler:awgdrill
- R11: value awgcurrent -> referenceopamp; footprint ece445_pcb:awgcurrent -> uiuc_ruler:referenceopamp
- R12: footprint ece445_pcb:logo -> uiuc_ruler:logo
- R15: footprint ece445_pcb:resistor -> uiuc_ruler:resistor
- R16: footprint ece445_pcb:referencebjt -> uiuc_ruler:referencebjt
- R17: footprint ece445_pcb:referencefet -> uiuc_ruler:referencefet
- R18: footprint ece445_pcb:referencediode -> uiuc_ruler:referencediode
- R19: footprint ece445_pcb:fontsize -> uiuc_ruler:fontsize
- R5: footprint ece445_pcb:rulerinches -> uiuc_ruler:rulerinches
- R6: footprint ece445_pcb:rulercm -> uiuc_ruler:rulercm
- R7: footprint ece445_pcb:traceswidths -> uiuc_ruler:traceswidths
- U11: value TO-252/DPAK -> TO-252
- U12: value QFP32 -> QFP-32
- U3: value SOT23-5 -> SOT-23-5
- U4: value SOT23-3 -> SOT-23-3
- U5: value SOT223 -> SOT-223
- U6: value SOIC20 -> SOIC-20
- U7: value TO220 -> TO-220; footprint ece445_pcb:TO-220-3_Vertical -> uiuc_ruler:TO-220-3_Vertical
- U8: value SOIC8 -> SOIC-8
- U9: value SOIC14 -> SOIC-14
Connections:
- net labels removed: +5V, GND, MISO, MOSI, SCK, ~RST
- wire segments 31 -> 0
Other:
- note added: "- crystals\n- dip"
- moved on the sheet: D10, D3, D4, D5, D6, D7, D8, D9, Q1, R10, R12, R13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
